File: new-joy-board/new-joy-board.sch (KiCad schematic (older format))
At the start: 3 parts, among them J1 Screw_Terminal_01x02, U1 AZReady_ESP32, U2 dc_dc_converter

Commit message: 3V3 power regulator and i2c0 bus
Parts:
- added D1: D, Diodes_THT:D_5KPW_P12.70mm_Horizontal, symbol D
- added J2: I2C_CONN, Pin_Headers:Pin_Header_Straight_1x04_Pitch2.54mm, symbol Conn_01x04
- added R1, R2: R, Resistors_THT:R_Axial_DIN0207_L6.3mm_D2.5mm_P2.54mm_Vertical, symbol R
- added U3: AZ1117-3.3, TO_SOT_Packages_SMD:SOT-223, symbol AZ1117-3.3
- renumbered U2 to U1, U1 to U2
Connections:
- net +5V: now also D1.1 (K), U3.3 (VI)
- net GND: now also J2.4 (Pin_4), U3.1 (GND)
- net SDA0: now reaches U2.12 (G14)
- net SDA0: now also J2.1 (Pin_1), R2.2
- net SCL0: now reaches U2.13 (G12)
- net SCL0: now also J2.3 (Pin_3), R1.2
- new net +3V3: D1.2 (A), J2.2 (Pin_2), R1.1, R2.1, U3.2 (VO)
Changed lines of the file:
@@
 $EndDescr
 $Comp
-L AZReady_ESP32 U1
+L AZReady_ESP32 U2
 U 1 1 5B23C3C4
 P 3650 3900
-F 0 "U1" H 3650 4900 50  0000 C CNN
+F 0 "U2" H 3650 4900 50  0000 C CNN
 F 1 "AZReady_ESP32" H 3650 2850 50  0000 C CNN
 F 2 "new-joy:AZReady_ESP32" H 3300 3900 50  0001 C CNN
@@
 $EndComp
 $Comp
-L GND #PWR01
+L GND #PWR9
 U 1 1 5B23D7F0
 P 3100 1500
-F 0 "#PWR01" H 3100 1250 50  0001 C CNN
+F 0 "#PWR9" H 3100 1250 50  0001 C CNN
 F 1 "GND" H 3100 1350 50  0000 C CNN
 F 2 "" H 3100 1500 50  0001 C CNN
@@
 $EndComp
 $Comp
-L +5V #PWR02
+L +5V #PWR8
 U 1 1 5B23DA07
 P 3100 1200
-F 0 "#PWR02" H 3100 1050 50  0001 C CNN
+F 0 "#PWR8" H 3100 1050 50  0001 C CNN
 F 1 "+5V" H 3100 1340 50  0000 C CNN
 F 2 "" H 3100 1200 50  0001 C CNN
@@
 $EndComp
 $Comp
-L dc_dc_converter U2
+L dc_dc_converter U1
 U 1 1 5B23E028
 P 2550 1350
-F 0 "U2" H 2550 1650 60  0000 C CNN
+F 0 "U1" H 2550 1650 60  0000 C CNN
 F 1 "dc_dc_converter" H 2550 1000 60  0000 C CNN
 F 2 "new-joy:dc_dc_converter" H 2550 1650 60  0001 C CNN
@@
 $EndComp
 $Comp
-L +5V #PWR03
+L +5V #PWR7
 U 1 1 5B2501A9
 P 2700 4800
-F 0 "#PWR03" H 2700 4650 50  0001 C CNN
+F 0 "#PWR7" H 2700 4650 50  0001 C CNN
 F 1 "+5V" H 2700 4940 50  0000 C CNN
 F 2 "" H 2700 4800 50  0001 C CNN
@@
 	2000 1600 2000 1500
 $Comp
-L GND #PWR04
+L GND #PWR10
 U 1 1 5B2501EA
 P 4750 3600
-F 0 "#PWR04" H 4750 3350 50  0001 C CNN
+F 0 "#PWR10" H 4750 3350 50  0001 C CNN
 F 1 "GND" H 4750 3450 50  0000 C CNN
 F 2 "" H 4750 3600 50  0001 C CNN
@@
 	4750 3000 4750 3600
 $Comp
-L +12V #PWR05
+L +12V #PWR3
 U 1 1 5B2502BB
 P 900 1050
-F 0 "#PWR05" H 900 900 50  0001 C CNN
+F 0 "#PWR3" H 900 900 50  0001 C CNN
 F 1 "+12V" H 900 1190 50  0000 C CNN
 F 2 "" H 900 1050 50  0001 C CNN
@@
 $EndComp
 $Comp
-L GNDPWR #PWR06
+L GNDPWR #PWR4
 U 1 1 5B2502FE
 P 900 1600
-F 0 "#PWR06" H 900 1400 50  0001 C CNN
+F 0 "#PWR4" H 900 1400 50  0001 C CNN
 F 1 "GNDPWR" H 900 1470 50  0000 C CNN
 F 2 "" H 900 1550 50  0001 C CNN
@@
 Wire Wire Line
 	2700 4800 3100 4800
+$Comp
+L AZ1117-3.3 U3
+U 1 1 5B250E5A
+P 9350 1200
+F 0 "U3" H 9200 1325 50  0000 C CNN
+F 1 "AZ1117-3.3" H 9350 1325 50  0000 L CNN
+F 2 "TO_SOT_Packages_SMD:SOT-223" H 9350 1450 50  0001 C CIN
+F 3 "" H 9350 1200 50  0001 C CNN
+	1    9350 1200
+	1    0    0    -1
+$EndComp
+$Comp
+L D D1
+U 1 1 5B25103F
+P 9350 850
+F 0 "D1" H 9350 950 50  0000 C CNN
+F 1 "D" H 9350 750 50  0000 C CNN
+F 2 "Diodes_THT:D_5KPW_P12.70mm_Horizontal" H 9350 850 50  0001 C CNN
+F 3 "" H 9350 850 50  0001 C CNN
+	1    9350 850
+	1    0    0    -1
+$EndComp
+Wire Wire Line
+	9650 1200 9650 850
+Wire Wire Line
+	9650 850  9500 850
+Wire Wire Line
+	9050 1200 9050 850
+Wire Wire Line
+	9050 850  9200 850
+$Comp
+L +5V #PWR11
+U 1 1 5B251122
+P 8900 1200
+F 0 "#PWR11" H 8900 1050 50  0001 C CNN
+F 1 "+5V" H 8900 1340 50  0000 C CNN
+F 2 "" H 8900 1200 50  0001 C CNN
+F 3 "" H 8900 1200 50  0001 C CNN
+	1    8900 1200
+	1    0    0    -1
+$EndComp
+$Comp
+L GND #PWR12
+U 1 1 5B251145
+P 9350 1500
+F 0 "#PWR12" H 9350 1250 50  0001 C CNN
+F 1 "GND" H 9350 1350 50  0000 C CNN
+F 2 "" H 9350 1500 50  0001 C CNN
+F 3 "" H 9350 1500 50  0001 C CNN
+	1    9350 1500
+	1    0    0    -1
+$EndComp
+$Comp
+L +3.3V #PWR13
+U 1 1 5B251203
+P 10000 1200
+F 0 "#PWR13" H 10000 1050 50  0001 C CNN
+F 1 "+3.3V" H 10000 1340 50  0000 C CNN
+F 2 "" H 10000 1200 50  0001 C CNN
+F 3 "" H 10000 1200 50  0001 C CNN
+	1    10000 1200
+	1    0    0    -1
+$EndComp
+Wire Wire Line
+	9650 1200 10000 1200
+Wire Wire Line
+	8900 1200 9050 1200
+Wire Wire Line
+	3100 4200 2650 4200
+Wire Wire Line
+	3100 4100 2650 4100
+Text Label 2650 4200 0    60   ~ 0
+SCL0
+Text Label 2650 4100 0    60   ~ 0
+SDA0
+$Comp
+L Conn_01x04 J2
+U 1 1 5B25176E
+P 1250 3150
+F 0 "J2" H 1250 3350 50  0000 C CNN
+F 1 "I2C_CONN" H 1250 2850 50  0000 C CNN
+F 2 "Pin_Headers:Pin_Header_Straight_1x04_Pitch2.54mm" H 1250 3150 50  0001 C CNN
+F 3 "" H 1250 3150 50  0001 C CNN
+	1    1250 3150
+	1    0    0    -1
+$EndComp
+Wire Wire Line
+	1050 3050 850  3050
+Wire Wire Line
+	1050 3150 700  3150
+Wire Wire Line
+	1050 3250 850  3250
+Wire Wire Line
+	1050 3350 700  3350
+Text Label 850  3050 0    60   ~ 0
+SDA0
+Text Label 850  3250 0    60   ~ 0
+SCL0
+$Comp
+L GND #PWR2
+U 1 1 5B251B24
+P 700 3350
+F 0 "#PWR2" H 700 3100 50  0001 C CNN
+F 1 "GND" H 700 3200 50  0000 C CNN
+F 2 "" H 700 3350 50  0001 C CNN
+F 3 "" H 700 3350 50  0001 C CNN
+	1    700  3350
+	1    0    0    -1
+$EndComp
+$Comp
+L +3.3V #PWR1
+U 1 1 5B251B4D
+P 700 3150
+F 0 "#PWR1" H 700 3000 50  0001 C CNN
+F 1 "+3.3V" H 700 3290 50  0000 C CNN
+F 2 "" H 700 3150 50  0001 C CNN
+F 3 "" H 700 3150 50  0001 C CNN
+	1    700  3150
+	1    0    0    -1
+$EndComp
+$Comp
+L R R1
+U 1 1 5B2525BD
+P 1800 3200
+F 0 "R1" V 1880 3200 50  0000 C CNN
+F 1 "R" V 1800 3200 50  0000 C CNN
+F 2 "Resistors_THT:R_Axial_DIN0207_L6.3mm_D2.5mm_P2.54mm_Vertical" V 1730 3200 50  0001 C CNN
+F 3 "" H 1800 3200 50  0001 C CNN
+	1    1800 3200
+	1    0    0    -1
+$EndComp
+$Comp
+L R R2
+U 1 1 5B25261D
+P 2100 3200
+F 0 "R2" V 2180 3200 50  0000 C CNN
+F 1 "R" V 2100 3200 50  0000 C CNN
+F 2 "Resistors_THT:R_Axial_DIN0207_L6.3mm_D2.5mm_P2.54mm_Vertical" V 2030 3200 50  0001 C CNN
+F 3 "" H 2100 3200 50  0001 C CNN
+	1    2100 3200
+	1    0    0    -1
+$EndComp
+Text Label 1800 3550 0    60   ~ 0
+SCL0
+Text Label 2100 3550 0    60   ~ 0
+SDA0
+Wire Wire Line
+	1800 3350 1800 3550
+Wire Wire Line
+	2100 3350 2100 3550
+$Comp
+L +3.3V #PWR5
+U 1 1 5B252734
+P 1800 3050
+F 0 "#PWR5" H 1800 2900 50  0001 C CNN
+F 1 "+3.3V" H 1800 3190 50  0000 C CNN
+F 2 "" H 1800 3050 50  0001 C CNN
+F 3 "" H 1800 3050 50  0001 C CNN
+	1    1800 3050
+	1    0    0    -1
+$EndComp
+$Comp
+L +3.3V #PWR6
+U 1 1 5B252763
+P 2100 3050
+F 0 "#PWR6" H 2100 2900 50  0001 C CNN
+F 1 "+3.3V" H 2100 3190 50  0000 C CNN
+F 2 "" H 2100 3050 50  0001 C CNN
+F 3 "" H 2100 3050 50  0001 C CNN
+	1    2100 3050
+	1    0    0    -1
+$EndComp
 $EndSCHEMATC

Commit message: Worked on design, including DMX and buffered I2C
Parts:
- added C1: 10uF, Capacitors_SMD:CP_Elec_5x5.3, symbol C
- added C2: 100nF, Capacitors_SMD:C_1210_HandSoldering, symbol C
- added J3: I2C_CONN_1, Pin_Headers:Pin_Header_Straight_1x04_Pitch2.54mm, symbol Conn_01x04
- added J4: I2C_CONN_2, Pin_Headers:Pin_Header_Straight_1x04_Pitch2.54mm, symbol Conn_01x04
- added J5: I2C_CONN_3, Pin_Headers:Pin_Header_Straight_1x04_Pitch2.54mm, symbol Conn_01x04
- added J6: DMX, Connectors_Terminal_Blocks:TerminalBlock_bornier-3_P5.08mm, symbol Screw_Terminal_01x03
- added R3: 133, Resistors_SMD:R_1210_HandSoldering, symbol R
- added RV1, RV2: 10K, Potentiometers:Potentiometer_Trimmer_Piher_PT-15v12.5_Horizontal_Px12.5mm_Py10.0mm, symbol POT_TRIM
- added U4: P82B715, new-joy:P82B715D, symbol P82B715
- added U5: MPU6050_Breakout, new-joy:MPU6050_Breakout, symbol MPU6050_Breakout
- added U6: MAX3072E, Housings_SOIC:SOIC-8_3.9x4.9mm_Pitch1.27mm, symbol MAX3072E
- J1: value Screw_Terminal_01x02 -> BAT
- J2: value I2C_CONN -> I2C_CONN_4
- R1, R2: value R -> 4K7; footprint Resistors_THT:R_Axial_DIN0207_L6.3mm_D2.5mm_P2.54mm_Vertical -> Resistors_SMD:R_1210_HandSoldering
Connections:
- net GNDPWR is gone; now on net GND: J1.2 (Pin_2), U1.2 (VIN-)
- net +3V3: now also C2.1, U5.1 (VCC), U6.2 (~RE~), U6.3 (DE), U6.8 (VCC); no longer J2.2 (Pin_2)
- net +5V: now also J2.2 (Pin_2), C1.1, J3.2 (Pin_2), J4.2 (Pin_2), J5.2 (Pin_2), RV1.1, RV2.1, U4.8 (VCC)
- net GND: now also C1.2, C2.2, J3.4 (Pin_4), J4.4 (Pin_4), J5.4 (Pin_4), J6.1 (Pin_1), U4.4 (GND), U5.2 (GND), U6.5 (GND)
- net at U2.35 (TXD): now also U6.4 (DI)
- net SCL0 renamed SCL0ESP
- net SCL0ESP: now also U4.6 (Sy), U5.3 (SCL); no longer J2.3 (Pin_3)
- net SDA0 renamed SDA0ESP
- net SDA0ESP: now also U4.3 (Sx), U5.4 (SDA); no longer J2.1 (Pin_1)
- new net: J6.2 (Pin_2), R3.1, U6.6 (A)
- new net: J6.3 (Pin_3), R3.2, U6.7 (B)
- new net SCL0BUF: J2.3 (Pin_3), J3.3 (Pin_3), J4.3 (Pin_3), J5.3 (Pin_3), RV1.3, U4.7 (Ly)
- new net SDA0BUF: J2.1 (Pin_1), J3.1 (Pin_1), J4.1 (Pin_1), J5.1 (Pin_1), RV2.3, U4.2 (Lx)
- no-connect marks 0 -> 5
Other:
- moved on the sheet: J1, J2, R1, R2, U1, U2

Commit message: Upgrade to kicad 5
Parts:
- C1, C2: symbol C -> new-joy-board-rescue:C
- D1: symbol D -> new-joy-board-rescue:D
- J1: symbol Screw_Terminal_01x02 -> new-joy-board-rescue:Screw_Terminal_01x02
- J2, J3, J4, J5: symbol Conn_01x04 -> new-joy-board-rescue:Conn_01x04
- J6: symbol Screw_Terminal_01x03 -> new-joy-board-rescue:Screw_Terminal_01x03
- R1, R2, R3: symbol R -> new-joy-board-rescue:R
- RV1, RV2: symbol POT_TRIM -> new-joy-board-rescue:POT_TRIM
- U1: symbol dc_dc_converter -> new-joy:dc_dc_converter
- U2: symbol AZReady_ESP32 -> new-joy:AZReady_ESP32
- U3: symbol AZ1117-3.3 -> new-joy-board-rescue:AZ1117-3.3
- U4: symbol P82B715 -> new-joy:P82B715
- U5: symbol MPU6050_Breakout -> new-joy:MPU6050_Breakout
- U6: symbol MAX3072E -> new-joy-board-rescue:MAX3072E
Changed lines of the file:
@@
-EESchema Schematic File Version 2
-LIBS:new-joy
-LIBS:power
-LIBS:device
-LIBS:transistors
-LIBS:conn
-LIBS:linear
-LIBS:regul
-LIBS:74xx
-LIBS:cmos4000
-LIBS:adc-dac
-LIBS:memory
-LIBS:xilinx
-LIBS:microcontrollers
-LIBS:dsp
-LIBS:microchip
-LIBS:analog_switches
-LIBS:motorola
-LIBS:texas
-LIBS:intel
-LIBS:audio
-LIBS:interface
-LIBS:digital-audio
-LIBS:philips
-LIBS:display
-LIBS:cypress
-LIBS:siliconi
-LIBS:opto
-LIBS:atmel
-LIBS:contrib
-LIBS:valves
+EESchema Schematic File Version 4
 LIBS:new-joy-board-cache
-EELAYER 25 0
+EELAYER 26 0
 EELAYER END
 $Descr A4 11693 8268
@@
 $EndDescr
 $Comp
-L AZReady_ESP32 U2
+L new-joy:AZReady_ESP32 U2
 U 1 1 5B23C3C4
 P 5600 3900
@@
 $EndComp
 $Comp
-L GND #PWR01
+L power:GND #PWR01
 U 1 1 5B23D7F0
 P 8400 1500
@@
 $EndComp
 $Comp
-L +5V #PWR02
+L power:+5V #PWR02
 U 1 1 5B23DA07
 P 8400 1200
@@
 $EndComp
 $Comp
-L dc_dc_converter U1
+L new-joy:dc_dc_converter U1
 U 1 1 5B23E028
 P 7850 1350
@@
 $EndComp
 $Comp
-L Screw_Terminal_01x02 J1
+L new-joy-board-rescue:Screw_Terminal_01x02 J1
 U 1 1 5B23E0D2
 P 6850 1300
@@
 $EndComp
 $Comp
-L +5V #PWR03
+L power:+5V #PWR03
 U 1 1 5B2501A9
 P 4650 4800
@@
 $EndComp
 $Comp
-L GND #PWR04
+L power:GND #PWR04
 U 1 1 5B2501EA
 P 6700 3600
@@
 $EndComp
 $Comp
-L +12V #PWR05
+L power:+12V #PWR05
 U 1 1 5B2502BB
 P 7050 1200
@@
 $EndComp
 $Comp
-L AZ1117-3.3 U3
+L new-joy-board-rescue:AZ1117-3.3 U3
 U 1 1 5B250E5A
 P 9350 1200
@@
 $EndComp
 $Comp
-L D D1
+L new-joy-board-rescue:D D1
 U 1 1 5B25103F
 P 9350 850
@@
 $EndComp
 $Comp
-L +5V #PWR07
+L power:+5V #PWR07
 U 1 1 5B251122
 P 8900 1200
@@
 $EndComp
 $Comp
-L GND #PWR08
+L power:GND #PWR08
 U 1 1 5B251145
 P 9350 1500
@@
 $EndComp
 $Comp
-L +3.3V #PWR09
+L power:+3.3V #PWR09
 U 1 1 5B251203
 P 10000 1200
@@
 SDA0ESP
 $Comp
-L Conn_01x04 J2
+L new-joy-board-rescue:Conn_01x04 J2
 U 1 1 5B25176E
 P 1750 6100
@@
 SCL0BUF
 $Comp
-L GND #PWR010
+L power:GND #PWR010
 U 1 1 5B251B24
 P 1050 6300
@@
 $EndComp
 $Comp
-L R R1
+L new-joy-board-rescue:R R1
 U 1 1 5B2525BD
 P 3950 3350
@@
 $EndComp
 $Comp
-L R R2
+L new-joy-board-rescue:R R2
 U 1 1 5B25261D
 P 3950 4150
@@
 SDA0ESP
 $Comp
-L +3.3V #PWR011
+L power:+3.3V #PWR011
 U 1 1 5B252734
 P 3950 3200
@@
 $EndComp
 $Comp
-L +3.3V #PWR012
+L power:+3.3V #PWR012
 U 1 1 5B252763
 P 3950 4000
@@
 $EndComp
 $Comp
-L MPU6050_Breakout U5
+L new-joy:MPU6050_Breakout U5
 U 1 1 5B25335B
 P 3850 5900
@@
 SDA0ESP
 $Comp
-L +3.3V #PWR013
+L power:+3.3V #PWR013
 U 1 1 5B25365F
 P 4650 5550
@@
 $EndComp
 $Comp
-L GND #PWR014
+L power:GND #PWR014
 U 1 1 5B25368E
 P 4650 5650
@@
 $EndComp
 $Comp
-L C C1
+L new-joy-board-rescue:C C1
 U 1 1 5B253942
 P 8900 1350
@@
 $EndComp
 $Comp
-L C C2
+L new-joy-board-rescue:C C2
 U 1 1 5B253992
 P 10000 1350
@@
 NoConn ~ 4000 5950
 $Comp
-L +5V #PWR015
+L power:+5V #PWR015
 U 1 1 5B2558CE
 P 1050 6100
@@
 $EndComp
 $Comp
-L P82B715 U4
+L new-joy:P82B715 U4
 U 1 1 5B2560BB
 P 3650 2250
@@
 $EndComp
 $Comp
-L +5V #PWR016
+L power:+5V #PWR016
 U 1 1 5B256249
 P 3250 2050
@@
 $EndComp
 $Comp
-L GND #PWR017
+L power:GND #PWR017
 U 1 1 5B256281
 P 4050 2350
@@
 SCL0ESP
 $Comp
-L +5V #PWR018
+L power:+5V #PWR018
 U 1 1 5B265432
 P 1300 900
@@
 $EndComp
 $Comp
-L +5V #PWR019
+L power:+5V #PWR019
 U 1 1 5B265470
 P 1300 1700
@@
 SDA0BUF
 $Comp
-L Conn_01x04 J5
+L new-joy-board-rescue:Conn_01x04 J5
 U 1 1 5B26748D
 P 1750 5100
@@
 SCL0BUF
 $Comp
-L GND #PWR020
+L power:GND #PWR020
 U 1 1 5B267499
 P 1050 5300
@@
 $EndComp
 $Comp
-L +5V #PWR021
+L power:+5V #PWR021
 U 1 1 5B26749F
 P 1050 5100
@@
 $EndComp
 $Comp
-L Conn_01x04 J4
+L new-joy-board-rescue:Conn_01x04 J4
 U 1 1 5B2674C8
 P 1750 4150
@@
 SCL0BUF
 $Comp
-L GND #PWR022
+L power:GND #PWR022
 U 1 1 5B2674D4
 P 1050 4350
@@
 $EndComp
 $Comp
-L +5V #PWR023
+L power:+5V #PWR023
 U 1 1 5B2674DA
 P 1050 4150
@@
 $EndComp
 $Comp
-L Conn_01x04 J3
+L new-joy-board-rescue:Conn_01x04 J3
 U 1 1 5B267501
 P 1750 3250
@@
 SCL0BUF
 $Comp
-L GND #PWR024
+L power:GND #PWR024
 U 1 1 5B26750D
 P 1050 3450
@@
 $EndComp
 $Comp
-L +5V #PWR025
+L power:+5V #PWR025
 U 1 1 5B267513
 P 1050 3250
@@
 $EndComp
 $Comp
-L MAX3072E U6
+L new-joy-board-rescue:MAX3072E U6
 U 1 1 5B268A5A
 P 8750 3850
@@
 $EndComp
 $Comp
-L +3V3 #PWR026
+L power:+3V3 #PWR026
 U 1 1 5B268E4C
 P 8750 3450
@@
 $EndComp
 $Comp
-L GND #PWR027
+L power:GND #PWR027
 U 1 1 5B268E96
 P 8750 4250
@@
 	4000 5550 4650 5550
 Wire Wire Line
-	8900 1500 10000 1500
+	8900 1500 9350 1500
 Connection ~ 9350 1500
 Wire Wire Line
@@
 	8350 3750 8350 3950
 $Comp
-L +3V3 #PWR028
+L power:+3V3 #PWR028
 U 1 1 5B2693C9
 P 8000 3950
@@
 	7350 4050 8350 4050
 $Comp
-L GND #PWR029
+L power:GND #PWR029
 U 1 1 5B26A7E9
 P 10000 4200
@@
 	10000 3750 10000 4200
 $Comp
-L R R3
+L new-joy-board-rescue:R R3
 U 1 1 5B26AB70
 P 9650 3900
@@
 $EndComp
 Wire Wire Line
-	9150 3750 9850 3750
+	9150 3750 9650 3750
 Wire Wire Line
 	9850 3750 9850 3850
@@
 	9400 3950 9400 4050
 Wire Wire Line
-	9400 4050 9850 4050
+	9400 4050 9650 4050
 Wire Wire Line
 	9850 4050 9850 3950
@@
 Connection ~ 9650 4050
 $Comp
-L Screw_Terminal_01x03 J6
+L new-joy-board-rescue:Screw_Terminal_01x03 J6
 U 1 1 5B26BC09
 P 10450 3850
@@
 $EndComp
 $Comp
-L POT_TRIM RV1
+L new-joy-board-rescue:POT_TRIM RV1
 U 1 1 5B26BF60
 P 1300 1050
@@
 $EndComp
 $Comp
-L POT_TRIM RV2
+L new-joy-board-rescue:POT_TRIM RV2
 U 1 1 5B26C0B7
 P 1300 1850
@@
 	1300 2000 1300 2100
 $Comp
-L GND #PWR?
+L power:GND #PWR?
 U 1 1 5B26B9FA
 P 7050 1500
@@
 	1    0    0    -1
 $EndComp
+Wire Wire Line
+	9350 1500 10000 1500
+Wire Wire Line
+	9650 3750 9850 3750
+Wire Wire Line
+	9650 4050 9850 4050
 $EndSCHEMATC
