File: new-joy-board/new-joy-board.sch (KiCad schematic (older format))
At the start: 20 parts, among them J1 BAT, J2 I2C_CONN_4, J3 I2C_CONN_1, J4 I2C_CONN_2, J5 I2C_CONN_3, J6 DMX, U1 dc_dc_converter, U2 AZReady_ESP32, U3 AZ1117-3.3, U4 P82B715, U5 MPU6050_Breakout, U6 MAX3072E

Commit message: Work on schematic and PCB to mock up real PCB
Parts:
- removed J2: I2C_CONN_4, Pin_Headers:Pin_Header_Straight_1x04_Pitch2.54mm, symbol Conn_01x04
- removed J3: I2C_CONN_1, Pin_Headers:Pin_Header_Straight_1x04_Pitch2.54mm, symbol Conn_01x04
- removed J4: I2C_CONN_2, Pin_Headers:Pin_Header_Straight_1x04_Pitch2.54mm, symbol Conn_01x04
- removed J5: I2C_CONN_3, Pin_Headers:Pin_Header_Straight_1x04_Pitch2.54mm, symbol Conn_01x04
- removed J6: DMX, Connectors_Terminal_Blocks:TerminalBlock_bornier-3_P5.08mm, symbol Screw_Terminal_01x03
- removed R3: 133, Resistors_SMD:R_1210_HandSoldering, symbol R
- removed RV1, RV2: 10K, Potentiometers:Potentiometer_Trimmer_Piher_PT-15v12.5_Horizontal_Px12.5mm_Py10.0mm, symbol POT_TRIM
- removed U6: MAX3072E, Housings_SOIC:SOIC-8_3.9x4.9mm_Pitch1.27mm, symbol MAX3072E
- added J0, J1, J2, J3: SDS-50J, new-joy:CUI_SDS-50J, symbol new-joy:SDS-50J
- added R10, R11, R12, R13, R14, R15, R16, R2, R4, R5, R6, R7, R8, R9: 4K7, Resistor_SMD:R_1210_3225Metric_Pad1.42x2.65mm_HandSolder, symbol new-joy-board-rescue:R
- added U0, U1, U2: P82B715, new-joy:P82B715D, symbol new-joy:P82B715
- C1: footprint Capacitors_SMD:CP_Elec_5x5.3 -> Capacitor_SMD:C_1210_3225Metric_Pad1.42x2.65mm_HandSolder; symbol C -> new-joy-board-rescue:C
- C2: footprint Capacitors_SMD:C_1210_HandSoldering -> Capacitor_SMD:C_1210_3225Metric_Pad1.42x2.65mm_HandSolder; symbol C -> new-joy-board-rescue:C
- D1: symbol D -> new-joy-board-rescue:D
- J4: renamed from J1; footprint Connectors_Terminal_Blocks:TerminalBlock_bornier-2_P5.08mm -> TerminalBlock:TerminalBlock_bornier-2_P5.08mm; symbol Screw_Terminal_01x02 -> new-joy-board-rescue:Screw_Terminal_01x02
- R1: footprint Resistors_SMD:R_1210_HandSoldering -> Resistor_SMD:R_1210_3225Metric_Pad1.42x2.65mm_HandSolder; symbol R -> new-joy-board-rescue:R
- R3: renamed from R2; footprint Resistors_SMD:R_1210_HandSoldering -> Resistor_SMD:R_1210_3225Metric_Pad1.42x2.65mm_HandSolder; symbol R -> new-joy-board-rescue:R
- U3: renamed from U4; symbol P82B715 -> new-joy:P82B715
- U4: renamed from U2; symbol AZReady_ESP32 -> new-joy:AZReady_ESP32
- U5: renamed from U1; symbol dc_dc_converter -> new-joy:dc_dc_converter
- U6: renamed from U3; footprint TO_SOT_Packages_SMD:SOT-223 -> Package_TO_SOT_SMD:SOT-223; symbol AZ1117-3.3 -> new-joy-board-rescue:AZ1117-3.3
- U7: renamed from U5; symbol MPU6050_Breakout -> new-joy:MPU6050_Breakout
Connections:
- net labels added: +BATT, -BATT, SCL1BUF, SCL1ESP, SCL2BUF, SCL2ESP, SCL3BUF, SCL3ESP, SDA1BUF, SDA1ESP, SDA2BUF, SDA2ESP, SDA3BUF, SDA3ESP
- net labels removed: +12V, +3V3
- wire segments 56 -> 51
- no-connect marks 5 -> 43
Other:
- moved on the sheet: R1, R3

Commit message: More PCB work to determine final dimensions for case construction
Parts:
- removed C1: 10uF, Capacitor_SMD:C_1210_3225Metric_Pad1.42x2.65mm_HandSolder, symbol new-joy-board-rescue:C
- removed C2: 100nF, Capacitor_SMD:C_1210_3225Metric_Pad1.42x2.65mm_HandSolder, symbol new-joy-board-rescue:C
- removed D1: D, Diodes_THT:D_5KPW_P12.70mm_Horizontal, symbol new-joy-board-rescue:D
- removed U6: AZ1117-3.3, Package_TO_SOT_SMD:SOT-223, symbol new-joy-board-rescue:AZ1117-3.3
Connections:
- wire segments 51 -> 43
- no-connect marks 43 -> 42
Changed lines of the file:
@@
-	1    0    0    -1
-$EndComp
-$Comp
-L new-joy-board-rescue:AZ1117-3.3 U6
-U 1 1 5B250E5A
-P 9350 1200
-F 0 "U6" H 9200 1325 50  0000 C CNN
-F 1 "AZ1117-3.3" H 9350 1325 50  0000 L CNN
-F 2 "Package_TO_SOT_SMD:SOT-223" H 9350 1450 50  0001 C CIN
-F 3 "" H 9350 1200 50  0001 C CNN
-	1    9350 1200
-	1    0    0    -1
-$EndComp
-$Comp
-L new-joy-board-rescue:D D1
-U 1 1 5B25103F
-P 9350 850
-F 0 "D1" H 9350 950 50  0000 C CNN
-F 1 "D" H 9350 750 50  0000 C CNN
-F 2 "Diodes_THT:D_5KPW_P12.70mm_Horizontal" H 9350 850 50  0001 C CNN
-F 3 "" H 9350 850 50  0001 C CNN
-	1    9350 850
-	1    0    0    -1
-$EndComp
-$Comp
-L power:+5V #PWR07
-U 1 1 5B251122
-P 8900 1200
-F 0 "#PWR07" H 8900 1050 50  0001 C CNN
-F 1 "+5V" H 8900 1340 50  0000 C CNN
-F 2 "" H 8900 1200 50  0001 C CNN
-F 3 "" H 8900 1200 50  0001 C CNN
-	1    8900 1200
-	1    0    0    -1
-$EndComp
-$Comp
-L power:GND #PWR08
-U 1 1 5B251145
-P 9350 1500
-F 0 "#PWR08" H 9350 1250 50  0001 C CNN
-F 1 "GND" H 9350 1350 50  0000 C CNN
-F 2 "" H 9350 1500 50  0001 C CNN
-F 3 "" H 9350 1500 50  0001 C CNN
-	1    9350 1500
-	1    0    0    -1
-$EndComp
-$Comp
-L power:+3.3V #PWR09
-U 1 1 5B251203
-P 10000 1200
-F 0 "#PWR09" H 10000 1050 50  0001 C CNN
-F 1 "+3.3V" H 10000 1340 50  0000 C CNN
-F 2 "" H 10000 1200 50  0001 C CNN
-F 3 "" H 10000 1200 50  0001 C CNN
-	1    10000 1200
 	1    0    0    -1
 $EndComp
@@
 	1    0    0    -1
 $EndComp
-$Comp
-L new-joy-board-rescue:C C1
-U 1 1 5B253942
-P 8900 1350
-F 0 "C1" H 8925 1450 50  0000 L CNN
-F 1 "10uF" H 8925 1250 50  0000 L CNN
-F 2 "Capacitor_SMD:C_1210_3225Metric_Pad1.42x2.65mm_HandSolder" H 8938 1200 50  0001 C CNN
-F 3 "" H 8900 1350 50  0001 C CNN
-	1    8900 1350
-	1    0    0    -1
-$EndComp
-$Comp
-L new-joy-board-rescue:C C2
-U 1 1 5B253992
-P 10000 1350
-F 0 "C2" H 10025 1450 50  0000 L CNN
-F 1 "100nF" H 10025 1250 50  0000 L CNN
-F 2 "Capacitor_SMD:C_1210_3225Metric_Pad1.42x2.65mm_HandSolder" H 10038 1200 50  0001 C CNN
-F 3 "" H 10000 1350 50  0001 C CNN
-	1    10000 1350
-	1    0    0    -1
-$EndComp
 NoConn ~ 9250 5850
 NoConn ~ 9250 5750
@@
 	4650 4800 5050 4800
 Wire Wire Line
-	9650 1200 9650 850
-Wire Wire Line
-	9650 850  9500 850
-Wire Wire Line
-	9050 1200 9050 850
-Wire Wire Line
-	9050 850  9200 850
-Wire Wire Line
-	9650 1200 10000 1200
-Wire Wire Line
-	8900 1200 9050 1200
-Wire Wire Line
 	5050 4200 4600 4200
 Wire Wire Line
@@
 Wire Wire Line
 	9250 5150 9900 5150
-Wire Wire Line
-	8900 1500 9350 1500
-Connection ~ 9350 1500
-Wire Wire Line
-	9350 1500 10000 1500
 Wire Wire Line
 	5050 4000 4600 4000
@@
 $EndComp
 Text Label 1650 1750 0    60   ~ 0
-SDA3ESP
+SDA3BUF
 Text Label 1650 2750 0    60   ~ 0
 SDA2BUF
@@
 $EndComp
 NoConn ~ 6200 3900
-NoConn ~ 5050 3000
 $Comp
 L new-joy:AZReady_ESP32 U4
@@
 	7050 1200 7300 1200
 $Comp
-L power:+5V #PWR?
+L power:+5V #PWR0108
 U 1 1 5B85BFDA
 P 1150 2000
-F 0 "#PWR?" H 1150 1850 50  0001 C CNN
+F 0 "#PWR0108" H 1150 1850 50  0001 C CNN
 F 1 "+5V" H 1165 2173 50  0000 C CNN
 F 2 "" H 1150 2000 50  0001 C CNN
@@
 $EndComp
 $Comp
-L power:+5V #PWR?
+L power:+5V #PWR0109
 U 1 1 5B85C05C
 P 900 2250
-F 0 "#PWR?" H 900 2100 50  0001 C CNN
+F 0 "#PWR0109" H 900 2100 50  0001 C CNN
 F 1 "+5V" H 915 2423 50  0000 C CNN
 F 2 "" H 900 2250 50  0001 C CNN
@@
 $EndComp
 $Comp
-L power:+5V #PWR?
+L power:+5V #PWR0110
 U 1 1 5B85C0DE
 P 900 1250
-F 0 "#PWR?" H 900 1100 50  0001 C CNN
+F 0 "#PWR0110" H 900 1100 50  0001 C CNN
 F 1 "+5V" H 915 1423 50  0000 C CNN
 F 2 "" H 900 1250 50  0001 C CNN
@@
 $EndComp
 $Comp
-L power:+5V #PWR?
+L power:+5V #PWR0111
 U 1 1 5B85C160
 P 1100 1000
-F 0 "#PWR?" H 1100 850 50  0001 C CNN
+F 0 "#PWR0111" H 1100 850 50  0001 C CNN
 F 1 "+5V" H 1115 1173 50  0000 C CNN
 F 2 "" H 1100 1000 50  0001 C CNN
@@
 $EndComp
 $Comp
-L power:+5V #PWR?
+L power:+5V #PWR0112
 U 1 1 5B85C1FE
 P 1850 1000
-F 0 "#PWR?" H 1850 850 50  0001 C CNN
+F 0 "#PWR0112" H 1850 850 50  0001 C CNN
 F 1 "+5V" H 1865 1173 50  0000 C CNN
 F 2 "" H 1850 1000 50  0001 C CNN
@@
 $EndComp
 $Comp
-L power:+5V #PWR?
+L power:+5V #PWR0113
 U 1 1 5B85C280
 P 1650 1250
-F 0 "#PWR?" H 1650 1100 50  0001 C CNN
+F 0 "#PWR0113" H 1650 1100 50  0001 C CNN
 F 1 "+5V" H 1665 1423 50  0000 C CNN
 F 2 "" H 1650 1250 50  0001 C CNN
@@
 $EndComp
 $Comp
-L power:+5V #PWR?
+L power:+5V #PWR0114
 U 1 1 5B85C302
 P 1900 2000
-F 0 "#PWR?" H 1900 1850 50  0001 C CNN
+F 0 "#PWR0114" H 1900 1850 50  0001 C CNN
 F 1 "+5V" H 1915 2173 50  0000 C CNN
 F 2 "" H 1900 2000 50  0001 C CNN
@@
 $EndComp
 $Comp
-L power:+5V #PWR?
+L power:+5V #PWR0115
 U 1 1 5B85C384
 P 1650 2250
-F 0 "#PWR?" H 1650 2100 50  0001 C CNN
+F 0 "#PWR0115" H 1650 2100 50  0001 C CNN
 F 1 "+5V" H 1665 2423 50  0000 C CNN
 F 2 "" H 1650 2250 50  0001 C CNN
@@
 	1    0    0    -1
 $EndComp
+$Comp
+L power:+3.3V #PWR0127
+U 1 1 5B81DEB8
+P 5050 3000
+F 0 "#PWR0127" H 5050 2850 50  0001 C CNN
+F 1 "+3.3V" H 5065 3173 50  0000 C CNN
+F 2 "" H 5050 3000 50  0001 C CNN
+F 3 "" H 5050 3000 50  0001 C CNN
+	1    5050 3000
+	1    0    0    -1
+$EndComp
+$Comp
+L power:+3.3V #PWR?
+U 1 1 5B81E2BA
+P 5350 1050
+F 0 "#PWR?" H 5350 900 50  0001 C CNN
+F 1 "+3.3V" H 5365 1223 50  0000 C CNN
+F 2 "" H 5350 1050 50  0001 C CNN
+F 3 "" H 5350 1050 50  0001 C CNN
+	1    5350 1050
+	1    0    0    -1
+$EndComp
+$Comp
+L power:PWR_FLAG #FLG?
+U 1 1 5B81E36F
+P 5350 1050
+F 0 "#FLG?" H 5350 1125 50  0001 C CNN
+F 1 "PWR_FLAG" H 5350 1223 50  0000 C CNN
+F 2 "" H 5350 1050 50  0001 C CNN
+F 3 "~" H 5350 1050 50  0001 C CNN
+	1    5350 1050
+	-1   0    0    1
+$EndComp
 $EndSCHEMATC

Commit message: Routet half of the I2C buffers
Parts:
- removed U5: dc_dc_converter, new-joy:dc_dc_converter, symbol new-joy:dc_dc_converter
- added U10: oskj-dc-dc, new-joy:oskj-dc-dc, symbol new-joy:oskj-dc-dc
Connections:
- wire segments 43 -> 47
- no-connect marks 42 -> 43
Changed lines of the file:
@@
 $EndDescr
-$Comp
-L power:GND #PWR01
-U 1 1 5B23D7F0
-P 8400 1500
-F 0 "#PWR01" H 8400 1250 50  0001 C CNN
-F 1 "GND" H 8400 1350 50  0000 C CNN
-F 2 "" H 8400 1500 50  0001 C CNN
-F 3 "" H 8400 1500 50  0001 C CNN
-	1    8400 1500
-	1    0    0    -1
-$EndComp
-$Comp
-L power:+5V #PWR02
-U 1 1 5B23DA07
-P 8400 1200
-F 0 "#PWR02" H 8400 1050 50  0001 C CNN
-F 1 "+5V" H 8400 1340 50  0000 C CNN
-F 2 "" H 8400 1200 50  0001 C CNN
-F 3 "" H 8400 1200 50  0001 C CNN
-	1    8400 1200
-	1    0    0    -1
-$EndComp
-$Comp
-L new-joy:dc_dc_converter U5
-U 1 1 5B23E028
-P 7850 1350
-F 0 "U5" H 7850 1650 60  0000 C CNN
-F 1 "dc_dc_converter" H 7850 1000 60  0000 C CNN
-F 2 "new-joy:dc_dc_converter" H 7850 1650 60  0001 C CNN
-F 3 "" H 7850 1650 60  0001 C CNN
-	1    7850 1350
-	1    0    0    -1
-$EndComp
 $Comp
 L new-joy-board-rescue:Screw_Terminal_01x02 J4
@@
 Wire Wire Line
 	7050 1400 7050 1500
-Wire Wire Line
-	7050 1500 7150 1500
 Wire Wire Line
 	6200 3600 6700 3600
@@
 NoConn ~ 6200 3300
 $Comp
-L power:+BATT #PWR0124
-U 1 1 5B85910A
-P 7150 1500
-F 0 "#PWR0124" H 7150 1350 50  0001 C CNN
-F 1 "+BATT" H 7165 1673 50  0000 C CNN
-F 2 "" H 7150 1500 50  0001 C CNN
-F 3 "" H 7150 1500 50  0001 C CNN
-	1    7150 1500
-	1    0    0    -1
-$EndComp
-Connection ~ 7150 1500
-Wire Wire Line
-	7150 1500 7300 1500
-$Comp
 L power:+BATT #PWR0123
 U 1 1 5B8598EF
@@
 	-1   0    0    1
 $EndComp
-$Comp
-L power:PWR_FLAG #FLG0102
-U 1 1 5B859ABC
-P 7050 1750
-F 0 "#FLG0102" H 7050 1825 50  0001 C CNN
-F 1 "PWR_FLAG" H 7050 1923 50  0000 C CNN
-F 2 "" H 7050 1750 50  0001 C CNN
-F 3 "~" H 7050 1750 50  0001 C CNN
-	1    7050 1750
-	-1   0    0    1
-$EndComp
-$Comp
-L power:-BATT #PWR0126
-U 1 1 5B859BE4
-P 7050 1750
-F 0 "#PWR0126" H 7050 1600 50  0001 C CNN
-F 1 "-BATT" H 7065 1923 50  0000 C CNN
-F 2 "" H 7050 1750 50  0001 C CNN
-F 3 "" H 7050 1750 50  0001 C CNN
-	1    7050 1750
-	1    0    0    -1
-$EndComp
 Wire Wire Line
 	7050 1200 7300 1200
@@
 $EndComp
 $Comp
-L power:+3.3V #PWR?
-U 1 1 5B81E2BA
-P 5350 1050
-F 0 "#PWR?" H 5350 900 50  0001 C CNN
-F 1 "+3.3V" H 5365 1223 50  0000 C CNN
-F 2 "" H 5350 1050 50  0001 C CNN
-F 3 "" H 5350 1050 50  0001 C CNN
-	1    5350 1050
-	1    0    0    -1
-$EndComp
-$Comp
-L power:PWR_FLAG #FLG?
+L power:PWR_FLAG #FLG0103
 U 1 1 5B81E36F
-P 5350 1050
-F 0 "#FLG?" H 5350 1125 50  0001 C CNN
-F 1 "PWR_FLAG" H 5350 1223 50  0000 C CNN
-F 2 "" H 5350 1050 50  0001 C CNN
-F 3 "~" H 5350 1050 50  0001 C CNN
-	1    5350 1050
+P 5350 1400
+F 0 "#FLG0103" H 5350 1475 50  0001 C CNN
+F 1 "PWR_FLAG" H 5350 1573 50  0000 C CNN
+F 2 "" H 5350 1400 50  0001 C CNN
+F 3 "~" H 5350 1400 50  0001 C CNN
+	1    5350 1400
+	1    0    0    -1
+$EndComp
+Wire Wire Line
+	7300 1200 7300 1400
+Wire Wire Line
+	7300 1400 7700 1400
+Wire Wire Line
+	7500 1500 7500 1300
+Wire Wire Line
+	7500 1300 7700 1300
+NoConn ~ 7700 1500
+$Comp
+L new-joy:oskj-dc-dc U10
+U 1 1 5B95549F
+P 8250 1350
+F 0 "U10" H 8627 1351 50  0000 L CNN
+F 1 "oskj-dc-dc" H 8627 1260 50  0000 L CNN
+F 2 "new-joy:oskj-dc-dc" H 8150 1250 50  0001 C CNN
+F 3 "" H 8250 1350 50  0001 C CNN
+	1    8250 1350
+	1    0    0    -1
+$EndComp
+$Comp
+L power:+5V #PWR0128
+U 1 1 5B95A721
+P 7700 1200
+F 0 "#PWR0128" H 7700 1050 50  0001 C CNN
+F 1 "+5V" H 7715 1373 50  0000 C CNN
+F 2 "" H 7700 1200 50  0001 C CNN
+F 3 "" H 7700 1200 50  0001 C CNN
+	1    7700 1200
+	1    0    0    -1
+$EndComp
+$Comp
+L power:GND #PWR0129
+U 1 1 5B95AAB2
+P 5350 1400
+F 0 "#PWR0129" H 5350 1150 50  0001 C CNN
+F 1 "GND" H 5355 1227 50  0000 C CNN
+F 2 "" H 5350 1400 50  0001 C CNN
+F 3 "" H 5350 1400 50  0001 C CNN
+	1    5350 1400
+	1    0    0    -1
+$EndComp
+$Comp
+L power:+3.3V #PWR0124
+U 1 1 5B95C2CE
+P 5350 850
+F 0 "#PWR0124" H 5350 700 50  0001 C CNN
+F 1 "+3.3V" H 5365 1023 50  0000 C CNN
+F 2 "" H 5350 850 50  0001 C CNN
+F 3 "" H 5350 850 50  0001 C CNN
+	1    5350 850
+	1    0    0    -1
+$EndComp
+$Comp
+L power:PWR_FLAG #FLG0104
+U 1 1 5B95C398
+P 5350 850
+F 0 "#FLG0104" H 5350 925 50  0001 C CNN
+F 1 "PWR_FLAG" H 5350 1023 50  0000 C CNN
+F 2 "" H 5350 850 50  0001 C CNN
+F 3 "~" H 5350 850 50  0001 C CNN
+	1    5350 850
 	-1   0    0    1
 $EndComp
+Wire Wire Line
+	7050 1500 7150 1500
+$Comp
+L power:-BATT #PWR0130
+U 1 1 5B95C876
+P 7150 1500
+F 0 "#PWR0130" H 7150 1350 50  0001 C CNN
+F 1 "-BATT" H 7165 1673 50  0000 C CNN
+F 2 "" H 7150 1500 50  0001 C CNN
+F 3 "" H 7150 1500 50  0001 C CNN
+	1    7150 1500
+	-1   0    0    1
+$EndComp
+$Comp
+L power:GND #PWR0131
+U 1 1 5B95FA7F
+P 7500 1500
+F 0 "#PWR0131" H 7500 1250 50  0001 C CNN
+F 1 "GND" H 7505 1327 50  0000 C CNN
+F 2 "" H 7500 1500 50  0001 C CNN
+F 3 "" H 7500 1500 50  0001 C CNN
+	1    7500 1500
+	1    0    0    -1
+$EndComp
+Connection ~ 7500 1500
+Connection ~ 7150 1500
+Wire Wire Line
+	7150 1500 7500 1500
 $EndSCHEMATC
