File: new-joy-board/bmp280-sensor-board/bmp280-sensor-board/bmp280-sensor-board.sch (KiCad schematic (older format))
At the start: 9 parts, among them J1 Conn_01x05, U1 TPS76933, U2 bmp280-board, U3 P82B715

Commit message: Placed MPU6050 as additional option
Parts:
- added R3, R4: 0K, Resistor_SMD:R_0805_2012Metric_Pad1.15x1.40mm_HandSolder, symbol Device:R
- added U4: MPU6050_Breakout, new-joy:MPU6050_Breakout, symbol new-joy:MPU6050_Breakout
Connections:
- no-connect marks 3 -> 5
Changed lines of the file:
@@
 Text Label 4200 3750 2    50   ~ 0
 SDA
-NoConn ~ 5400 3550
 NoConn ~ 5400 3750
 $Comp
@@
 Wire Wire Line
 	5650 3500 6500 3500
+$Comp
+L new-joy:MPU6050_Breakout U4
+U 1 1 5BAF5DE9
+P 4800 5600
+F 0 "U4" H 4800 6250 60  0000 C CNN
+F 1 "MPU6050_Breakout" H 4800 6144 60  0000 C CNN
+F 2 "new-joy:MPU6050_Breakout" H 4750 6300 60  0001 C CNN
+F 3 "" H 4250 5450 60  0001 C CNN
+	1    4800 5600
+	1    0    0    -1
+$EndComp
+$Comp
+L power:+3.3V #PWR013
+U 1 1 5BAF5E77
+P 4800 5150
+F 0 "#PWR013" H 4800 5000 50  0001 C CNN
+F 1 "+3.3V" H 4815 5323 50  0000 C CNN
+F 2 "" H 4800 5150 50  0001 C CNN
+F 3 "" H 4800 5150 50  0001 C CNN
+	1    4800 5150
+	1    0    0    -1
+$EndComp
+$Comp
+L power:GND #PWR014
+U 1 1 5BAF5EF6
+P 4800 6000
+F 0 "#PWR014" H 4800 5750 50  0001 C CNN
+F 1 "GND" H 4805 5827 50  0000 C CNN
+F 2 "" H 4800 6000 50  0001 C CNN
+F 3 "" H 4800 6000 50  0001 C CNN
+	1    4800 6000
+	1    0    0    -1
+$EndComp
+Text Label 5250 5500 0    50   ~ 0
+SCL
+Text Label 5250 5600 0    50   ~ 0
+SDA
+NoConn ~ 5250 5700
+NoConn ~ 4350 5600
+NoConn ~ 4350 5500
+$Comp
+L Device:R R3
+U 1 1 5BAF5DA2
+P 4200 5700
+F 0 "R3" V 3993 5700 50  0000 C CNN
+F 1 "0K" V 4084 5700 50  0000 C CNN
+F 2 "Resistor_SMD:R_0805_2012Metric_Pad1.15x1.40mm_HandSolder" V 4130 5700 50  0001 C CNN
+F 3 "~" H 4200 5700 50  0001 C CNN
+	1    4200 5700
+	0    1    1    0
+$EndComp
+$Comp
+L power:+3.3V #PWR015
+U 1 1 5BAF5E16
+P 4050 5700
+F 0 "#PWR015" H 4050 5550 50  0001 C CNN
+F 1 "+3.3V" H 4065 5873 50  0000 C CNN
+F 2 "" H 4050 5700 50  0001 C CNN
+F 3 "" H 4050 5700 50  0001 C CNN
+	1    4050 5700
+	1    0    0    -1
+$EndComp
+$Comp
+L Device:R R4
+U 1 1 5BAF5F95
+P 5400 3400
+F 0 "R4" H 5470 3446 50  0000 L CNN
+F 1 "0K" H 5470 3355 50  0000 L CNN
+F 2 "Resistor_SMD:R_0805_2012Metric_Pad1.15x1.40mm_HandSolder" V 5330 3400 50  0001 C CNN
+F 3 "~" H 5400 3400 50  0001 C CNN
+	1    5400 3400
+	1    0    0    -1
+$EndComp
+$Comp
+L power:+3.3V #PWR016
+U 1 1 5BAF5FF7
+P 5400 3250
+F 0 "#PWR016" H 5400 3100 50  0001 C CNN
+F 1 "+3.3V" H 5415 3423 50  0000 C CNN
+F 2 "" H 5400 3250 50  0001 C CNN
+F 3 "" H 5400 3250 50  0001 C CNN
+	1    5400 3250
+	1    0    0    -1
+$EndComp
 $EndSCHEMATC
