File: new-joy-board/bmp280-sensor-board/bmp280-sensor-board.sch (KiCad schematic (older format))
At the start: 12 parts, among them J1 Conn_01x05, U1 TPS76933, U2 bmp280-board, U3 P82B715, U4 MPU6050_Breakout

Commit message: Continue work on daughter board
Parts:
- removed R3, R4: 0K, Resistor_SMD:R_0805_2012Metric_Pad1.15x1.40mm_HandSolder, symbol Device:R
- removed U2: bmp280-board, new-joy:bmp280-board-footprint, symbol new-joy:bmp280-board
- removed U4: MPU6050_Breakout, new-joy:MPU6050_Breakout, symbol new-joy:MPU6050_Breakout
- added J2: Conn_01x05, Connector_PinHeader_2.54mm:PinHeader_1x05_P2.54mm_Vertical, symbol Connector_Generic:Conn_01x05
- added U2, U4: generic-i2c-device, new-joy:generic-i2c-device, symbol new-joy:generic-i2c-device
- J1: footprint Connector_PinHeader_2.54mm:PinHeader_1x05_P2.54mm_Horizontal -> Connector_PinHeader_2.54mm:PinHeader_1x05_P2.54mm_Vertical
Connections:
- wire segments 16 -> 19
- no-connect marks 5 -> 2
Changed lines of the file:
@@
 $EndDescr
-$Comp
-L new-joy:bmp280-board U2
-U 1 1 5BAE3021
-P 4800 3650
-F 0 "U2" H 4800 4278 50  0000 C CNN
-F 1 "bmp280-board" H 4800 4187 50  0000 C CNN
-F 2 "new-joy:bmp280-board-footprint" H 4700 3650 50  0001 C CNN
-F 3 "" H 4800 3650 50  0001 C CNN
-	1    4800 3650
-	1    0    0    -1
-$EndComp
 $Comp
 L Regulator_Linear:TPS76933 U1
@@
 $EndComp
 Connection ~ 3550 3600
-$Comp
-L power:GND #PWR05
-U 1 1 5BAE39E6
-P 4800 4100
-F 0 "#PWR05" H 4800 3850 50  0001 C CNN
-F 1 "GND" H 4805 3927 50  0000 C CNN
-F 2 "" H 4800 4100 50  0001 C CNN
-F 3 "" H 4800 4100 50  0001 C CNN
-	1    4800 4100
-	1    0    0    -1
-$EndComp
-$Comp
-L power:+3.3V #PWR04
-U 1 1 5BAE3A4D
-P 4800 2850
-F 0 "#PWR04" H 4800 2700 50  0001 C CNN
-F 1 "+3.3V" H 4815 3023 50  0000 C CNN
-F 2 "" H 4800 2850 50  0001 C CNN
-F 3 "" H 4800 2850 50  0001 C CNN
-	1    4800 2850
-	1    0    0    -1
-$EndComp
-Wire Wire Line
-	4800 3200 4800 2850
 Text Label 4200 3550 2    50   ~ 0
 SCL
 Text Label 4200 3750 2    50   ~ 0
 SDA
-NoConn ~ 5400 3750
 $Comp
 L new-joy:P82B715 U3
@@
 F 0 "J1" H 8130 3692 50  0000 L CNN
 F 1 "Conn_01x05" H 8130 3601 50  0000 L CNN
-F 2 "Connector_PinHeader_2.54mm:PinHeader_1x05_P2.54mm_Horizontal" H 8050 3650 50  0001 C CNN
+F 2 "Connector_PinHeader_2.54mm:PinHeader_1x05_P2.54mm_Vertical" H 8050 3650 50  0001 C CNN
 F 3 "~" H 8050 3650 50  0001 C CNN
 	1    8050 3650
@@
 	5650 3500 6500 3500
 $Comp
-L new-joy:MPU6050_Breakout U4
-U 1 1 5BAF5DE9
-P 4800 5600
-F 0 "U4" H 4800 6250 60  0000 C CNN
-F 1 "MPU6050_Breakout" H 4800 6144 60  0000 C CNN
-F 2 "new-joy:MPU6050_Breakout" H 4750 6300 60  0001 C CNN
-F 3 "" H 4250 5450 60  0001 C CNN
-	1    4800 5600
+L new-joy:generic-i2c-device U4
+U 1 1 5BB4E3D6
+P 5800 4950
+F 0 "U4" H 6077 4996 50  0000 L CNN
+F 1 "generic-i2c-device" H 6077 4905 50  0000 L CNN
+F 2 "new-joy:generic-i2c-device" H 5800 4950 50  0001 C CNN
+F 3 "" H 5800 4950 50  0001 C CNN
+	1    5800 4950
 	1    0    0    -1
 $EndComp
 $Comp
 L power:+3.3V #PWR013
-U 1 1 5BAF5E77
-P 4800 5150
-F 0 "#PWR013" H 4800 5000 50  0001 C CNN
-F 1 "+3.3V" H 4815 5323 50  0000 C CNN
-F 2 "" H 4800 5150 50  0001 C CNN
-F 3 "" H 4800 5150 50  0001 C CNN
-	1    4800 5150
+U 1 1 5BB4E4D4
+P 5800 4600
+F 0 "#PWR013" H 5800 4450 50  0001 C CNN
+F 1 "+3.3V" H 5815 4773 50  0000 C CNN
+F 2 "" H 5800 4600 50  0001 C CNN
+F 3 "" H 5800 4600 50  0001 C CNN
+	1    5800 4600
 	1    0    0    -1
 $EndComp
 $Comp
 L power:GND #PWR014
-U 1 1 5BAF5EF6
-P 4800 6000
-F 0 "#PWR014" H 4800 5750 50  0001 C CNN
-F 1 "GND" H 4805 5827 50  0000 C CNN
-F 2 "" H 4800 6000 50  0001 C CNN
-F 3 "" H 4800 6000 50  0001 C CNN
-	1    4800 6000
-	1    0    0    -1
-$EndComp
-Text Label 5250 5500 0    50   ~ 0
+U 1 1 5BB4E550
+P 5800 5300
+F 0 "#PWR014" H 5800 5050 50  0001 C CNN
+F 1 "GND" H 5805 5127 50  0000 C CNN
+F 2 "" H 5800 5300 50  0001 C CNN
+F 3 "" H 5800 5300 50  0001 C CNN
+	1    5800 5300
+	1    0    0    -1
+$EndComp
+Text Label 5250 5000 0    50   ~ 0
+SDA
+Text Label 5250 4900 0    50   ~ 0
 SCL
-Text Label 5250 5600 0    50   ~ 0
+Wire Wire Line
+	5450 5000 5250 5000
+Wire Wire Line
+	5450 4900 5250 4900
+$Comp
+L new-joy:generic-i2c-device U2
+U 1 1 5BB4EE93
+P 3850 5000
+F 0 "U2" H 4127 5046 50  0000 L CNN
+F 1 "generic-i2c-device" H 4127 4955 50  0000 L CNN
+F 2 "new-joy:generic-i2c-device" H 3850 5000 50  0001 C CNN
+F 3 "" H 3850 5000 50  0001 C CNN
+	1    3850 5000
+	1    0    0    -1
+$EndComp
+$Comp
+L power:+3.3V #PWR04
+U 1 1 5BB4EE9A
+P 3850 4650
+F 0 "#PWR04" H 3850 4500 50  0001 C CNN
+F 1 "+3.3V" H 3865 4823 50  0000 C CNN
+F 2 "" H 3850 4650 50  0001 C CNN
+F 3 "" H 3850 4650 50  0001 C CNN
+	1    3850 4650
+	1    0    0    -1
+$EndComp
+$Comp
+L power:GND #PWR05
+U 1 1 5BB4EEA0
+P 3850 5350
+F 0 "#PWR05" H 3850 5100 50  0001 C CNN
+F 1 "GND" H 3855 5177 50  0000 C CNN
+F 2 "" H 3850 5350 50  0001 C CNN
+F 3 "" H 3850 5350 50  0001 C CNN
+	1    3850 5350
+	1    0    0    -1
+$EndComp
+Text Label 3300 5050 0    50   ~ 0
 SDA
-NoConn ~ 5250 5700
-NoConn ~ 4350 5600
-NoConn ~ 4350 5500
-$Comp
-L Device:R R3
-U 1 1 5BAF5DA2
-P 4200 5700
-F 0 "R3" V 3993 5700 50  0000 C CNN
-F 1 "0K" V 4084 5700 50  0000 C CNN
-F 2 "Resistor_SMD:R_0805_2012Metric_Pad1.15x1.40mm_HandSolder" V 4130 5700 50  0001 C CNN
-F 3 "~" H 4200 5700 50  0001 C CNN
-	1    4200 5700
-	0    1    1    0
-$EndComp
-$Comp
-L power:+3.3V #PWR015
-U 1 1 5BAF5E16
-P 4050 5700
-F 0 "#PWR015" H 4050 5550 50  0001 C CNN
-F 1 "+3.3V" H 4065 5873 50  0000 C CNN
-F 2 "" H 4050 5700 50  0001 C CNN
-F 3 "" H 4050 5700 50  0001 C CNN
-	1    4050 5700
-	1    0    0    -1
-$EndComp
-$Comp
-L Device:R R4
-U 1 1 5BAF5F95
-P 5400 3400
-F 0 "R4" H 5470 3446 50  0000 L CNN
-F 1 "0K" H 5470 3355 50  0000 L CNN
-F 2 "Resistor_SMD:R_0805_2012Metric_Pad1.15x1.40mm_HandSolder" V 5330 3400 50  0001 C CNN
-F 3 "~" H 5400 3400 50  0001 C CNN
-	1    5400 3400
-	1    0    0    -1
-$EndComp
-$Comp
-L power:+3.3V #PWR016
-U 1 1 5BAF5FF7
-P 5400 3250
-F 0 "#PWR016" H 5400 3100 50  0001 C CNN
-F 1 "+3.3V" H 5415 3423 50  0000 C CNN
-F 2 "" H 5400 3250 50  0001 C CNN
-F 3 "" H 5400 3250 50  0001 C CNN
-	1    5400 3250
-	1    0    0    -1
-$EndComp
+Text Label 3300 4950 0    50   ~ 0
+SCL
+Wire Wire Line
+	3500 5050 3300 5050
+Wire Wire Line
+	3500 4950 3300 4950
+$Comp
+L Connector_Generic:Conn_01x05 J2
+U 1 1 5BB51A60
+P 8050 4650
+F 0 "J2" H 8130 4692 50  0000 L CNN
+F 1 "Conn_01x05" H 8130 4601 50  0000 L CNN
+F 2 "Connector_PinHeader_2.54mm:PinHeader_1x05_P2.54mm_Vertical" H 8050 4650 50  0001 C CNN
+F 3 "~" H 8050 4650 50  0001 C CNN
+	1    8050 4650
+	-1   0    0    1
+$EndComp
+$Comp
+L power:GND #PWR?
+U 1 1 5BB51A67
+P 8250 4850
+F 0 "#PWR?" H 8250 4600 50  0001 C CNN
+F 1 "GND" H 8255 4677 50  0000 C CNN
+F 2 "" H 8250 4850 50  0001 C CNN
+F 3 "" H 8250 4850 50  0001 C CNN
+	1    8250 4850
+	1    0    0    -1
+$EndComp
+$Comp
+L power:+5V #PWR?
+U 1 1 5BB51A6D
+P 8250 4450
+F 0 "#PWR?" H 8250 4300 50  0001 C CNN
+F 1 "+5V" H 8265 4623 50  0000 C CNN
+F 2 "" H 8250 4450 50  0001 C CNN
+F 3 "" H 8250 4450 50  0001 C CNN
+	1    8250 4450
+	1    0    0    -1
+$EndComp
+NoConn ~ 8250 4750
+Text Label 8250 4650 0    50   ~ 0
+SCLBUF
+Text Label 8250 4550 0    50   ~ 0
+SDABUF
 $EndSCHEMATC

Commit message: Prolonged daughter board and added footprint for better soldering
Parts:
- J1, J2: footprint Connector_PinHeader_2.54mm:PinHeader_1x05_P2.54mm_Vertical -> new-joy:Buffered-I2C-Cable-Connector
Changed lines of the file:
@@
 F 0 "J1" H 8130 3692 50  0000 L CNN
 F 1 "Conn_01x05" H 8130 3601 50  0000 L CNN
-F 2 "Connector_PinHeader_2.54mm:PinHeader_1x05_P2.54mm_Vertical" H 8050 3650 50  0001 C CNN
+F 2 "new-joy:Buffered-I2C-Cable-Connector" H 8050 3650 50  0001 C CNN
 F 3 "~" H 8050 3650 50  0001 C CNN
 	1    8050 3650
@@
 F 0 "J2" H 8130 4692 50  0000 L CNN
 F 1 "Conn_01x05" H 8130 4601 50  0000 L CNN
-F 2 "Connector_PinHeader_2.54mm:PinHeader_1x05_P2.54mm_Vertical" H 8050 4650 50  0001 C CNN
+F 2 "new-joy:Buffered-I2C-Cable-Connector" H 8050 4650 50  0001 C CNN
 F 3 "~" H 8050 4650 50  0001 C CNN
 	1    8050 4650
@@
 $EndComp
 $Comp
-L power:GND #PWR?
+L power:GND #PWR0101
 U 1 1 5BB51A67
 P 8250 4850
-F 0 "#PWR?" H 8250 4600 50  0001 C CNN
+F 0 "#PWR0101" H 8250 4600 50  0001 C CNN
 F 1 "GND" H 8255 4677 50  0000 C CNN
 F 2 "" H 8250 4850 50  0001 C CNN
@@
 $EndComp
 $Comp
-L power:+5V #PWR?
+L power:+5V #PWR0102
 U 1 1 5BB51A6D
 P 8250 4450
-F 0 "#PWR?" H 8250 4300 50  0001 C CNN
+F 0 "#PWR0102" H 8250 4300 50  0001 C CNN
 F 1 "+5V" H 8265 4623 50  0000 C CNN
 F 2 "" H 8250 4450 50  0001 C CNN
